File: MeshDeck/MeshDeck.kicad_pcb (KiCad board)
At the start: 4 copper layers, 87 x 111.5 mm, 236 parts, among them CN1 ATGM336H-6N-74, J1 Conn_01x03_MountingPin, J2 Conn_02x05_Odd_Even, J3 Conn_02x08_Odd_Even, SW1 4*4*1.7, SW10 4*4*1.7, SW11 4*4*1.7, SW12 4*4*1.7, SW13 4*4*1.7, SW14 4*4*1.7, SW15 4*4*1.7, SW16 4*4*1.7, SW17 4*4*1.7, SW18 4*4*1.7, SW19 4*4*1.7, SW2 4*4*1.7, SW20 4*4*1.7, SW21 4*4*1.7, SW22 4*4*1.7, SW23 4*4*1.7, SW24 4*4*1.7, SW25 4*4*1.7, SW26 4*4*1.7, SW27 4*4*1.7, SW28 4*4*1.7, SW29 4*4*1.7, SW3 SKHHLVA010, SW30 4*4*1.7, SW31 4*4*1.7, SW32 4*4*1.7, SW33 4*4*1.7, SW34 4*4*1.7, SW35 4*4*1.7, SW36 4*4*1.7, SW37 4*4*1.7, SW38 4*4*1.7, SW39 4*4*1.7, SW4 4*4*1.7, SW5 4*4*1.7, SW6 4*4*1.7, SW7 4*4*1.7, SW8 4*4*1.7, SW9 4*4*1.7, U1 ESP32-S3-WROOM-1U-N16R8, U10 ABM8-272-T3_C20625731, U2 SX1262S8S+T-X1, U3 TPS6282533DMQR, U4 BQ24074RGTR, U5 RN32768114, U7 CD4013BM, U8 RP2040, U9 W25Q128JVSIQTR

Commit message: Wired kb matrix
Parts:
- moved C32 63.7 mm to (113.8, 66.1), turned to 180 degrees
- moved U9 62.5 mm to (120.2, 68.1), turned to -90 degrees
- moved C34 58.7 mm to (113.3, 69.6), turned to 0 degrees
- moved C26 55.6 mm to (121.5, 73.6), turned to 90 degrees
- moved R26 54.9 mm to (116.0, 72.7), turned to -90 degrees
- moved C23 54.6 mm to (118.8, 73.6), turned to 90 degrees
- moved U10 54.5 mm to (113.2, 72.6), turned to 90 degrees
- moved C24 54.1 mm to (117.5, 73.6), turned to 90 degrees
- moved C21 49.8 mm to (124.8, 79.4), turned to 180 degrees
- moved C30 47.1 mm to (113.0, 77.9), turned to 180 degrees
- moved U8 45.9 mm to (119.0, 80.0), turned to 90 degrees
- moved C28 45.7 mm to (124.8, 82.6), turned to 0 degrees
- moved C29 45.3 mm to (113.0, 79.1), turned to 0 degrees
- moved D20 45.2 mm to (171.1, 117.5)
- moved D18 45.2 mm to (153.4, 117.5)
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Routing:
- net /Keyboard/ROW2: track 0.00 -> 103.5 mm
- net /Keyboard/ROW1: track 0.00 -> 103.2 mm
- net /Keyboard/ROW3: track 0.00 -> 103.2 mm
- net /Keyboard/COL9: track 0.00 -> 66.8 mm, vias 0 -> 7
- net /Keyboard/COL4: track 0.00 -> 66.0 mm, vias 0 -> 7
- net /Keyboard/COL8: track 0.00 -> 65.3 mm, vias 0 -> 7
- net /Keyboard/ROW4: track 0.00 -> 58.5 mm
- net /Keyboard/COL5: track 0.00 -> 57.5 mm, vias 0 -> 2
- net /Keyboard/COL6: track 0.00 -> 57.4 mm, vias 0 -> 7
- net /Keyboard/COL7: track 0.00 -> 57.3 mm, vias 0 -> 7
- net /Keyboard/COL10: track 0.00 -> 50.0 mm, vias 0 -> 6
- net /Keyboard/COL2: track 0.00 -> 45.4 mm, vias 0 -> 6
- net /Keyboard/COL3: track 0.00 -> 44.7 mm, vias 0 -> 6
- net /Keyboard/COL1: track 0.00 -> 43.9 mm, vias 0 -> 6
- net Net-(CN1-RF_IN): track 0.00 -> 7.16 mm
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Other:
- board size 87 x 111.5 mm -> 88.9 x 121.6 mm

Commit message: More routing
Parts:
- moved C33 39.8 mm to (110.0, 72.7)
- moved R5 16.0 mm to (177.2, 87.0)
- moved C5 15.6 mm to (177.2, 85.5)
- moved R6 15.6 mm to (177.4, 89.5)
- moved D1 14.5 mm to (172.8, 87.5), turned to 180 degrees
- moved R10 8.68 mm to (154.5, 92.5), turned to 90 degrees
- moved C6 8.53 mm to (155.8, 92.5), turned to -90 degrees
- moved C7 7.39 mm to (152.0, 89.8), turned to 0 degrees
- moved R9 6.71 mm to (152.0, 88.3)
- moved C8 6.52 mm to (156.0, 85.0), turned to 90 degrees
- moved R11 6.48 mm to (154.8, 85.1), turned to -90 degrees
- moved C15 5.79 mm to (157.4, 79.0)
- moved C14 5.11 mm to (157.4, 73.0)
- moved J1 2.41 mm to (107.0, 148.9)
- moved U4 1.52 mm to (155.5, 89.0), turned to -90 degrees
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Connections:
- CN1 pad 2: /LORA_CS -> /RXD0_ESP
- CN1 pad 3: /LORA_CS -> /RXD0_ESP
- U1 pad 36: /LORA_CS -> /RXD0_ESP
- U1 pad 37: /LORA_CS -> /RXD0_ESP
Routing:
- net /Power Sheet/BCC_OUT: track 0.00 -> 109.7 mm, vias 0 -> 4
- net Net-(J1-Pin_1): track 0.00 -> 98.1 mm, vias 0 -> 2
- net Net-(J1-Pin_3): track 0.00 -> 92.6 mm, vias 0 -> 2
- net /3V3: track 3.60 -> 78.6 mm
- net /LORA_TXEN: track 0.00 -> 72.0 mm
- net Net-(LED2-K): track 0.00 -> 66.2 mm, vias 0 -> 4
- net Net-(LED3-A): track 0.00 -> 57.9 mm
- net Net-(LED4-A): track 0.00 -> 56.0 mm
- net /LORA_BUSY: track 0.00 -> 55.1 mm, vias 0 -> 2
- net /LORA_DIO1: track 0.50 -> 52.6 mm
- net /Power Sheet/CLOCK1: track 0.00 -> 45.6 mm
- net /USBSheet/VBUS: track 0.00 -> 44.3 mm, vias 0 -> 2
- net Net-(LED1-K): track 0.00 -> 44.3 mm, vias 0 -> 2
- net /SPI.MISO: track 0.00 -> 36.1 mm
- net /LORA_CS: track 0.00 -> 35.0 mm
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
Commit message: Too much routing
Parts:
- removed J2: Conn_02x05_Odd_Even, Connector_PinSocket_2.54mm:PinSocket_2x05_P2.54mm_Horizontal
- removed J3: Conn_02x08_Odd_Even, Connector_PinSocket_2.54mm:PinSocket_2x08_P2.54mm_Horizontal
- moved C16 4.00 mm to (116.4, 36.1)
- moved C17 4.00 mm to (117.7, 36.1)
- moved U2 4.00 mm to (116.0, 47.0)
- moved U6 3.76 mm to (120.2, 72.0)
- moved C27 1.80 mm to (119.2, 87.2), turned to 0 degrees
- moved C25 1.49 mm to (122.5, 84.8), turned to 0 degrees
- moved R2 1.01 mm to (140.0, 87.6)
- moved R13 0.96 mm to (131.9, 88.2), turned to -90 degrees
- moved C5 0.71 mm to (177.8, 85.0), turned to 90 degrees
- moved C23 0.65 mm to (119.4, 73.6)
- moved C24 0.65 mm to (118.2, 73.6)
- moved R5 0.27 mm to (177.0, 86.9)
- moved R51 0.25 mm to (139.0, 127.1)
Connections:
- net /IO10 renamed /SCR_RESET
- net /IO11 renamed /SCR_CD
- net /IO42 renamed /SCR_LED
- net /IO48 renamed /GPS_EN
- CN1 pad 3: /RXD0_ESP -> /TXD0_ESP
- U1 pad 37: /RXD0_ESP -> /TXD0_ESP
- U8 pad 2: /Keyboard/GPBOOT -> /Keyboard/GPIO0
- U8 pad 32: /Keyboard/GPTCH_CS -> /Keyboard/GPIO21
- U8 pad 5: /Keyboard/GPGPS_PPS -> /Keyboard/GPIO3
Routing:
- net /3V3: track 78.6 -> 316.7 mm, vias 0 -> 6
- net /Keyboard/ROW4: track 58.5 -> 172.9 mm, vias 0 -> 1
- net /Keyboard/ROW3: track 103.2 -> 181.5 mm, vias 0 -> 1
- net /Keyboard/COL9: track 66.8 -> 144.1 mm, vias 7 -> 9
- net /Keyboard/COL10: track 50.0 -> 124.7 mm, vias 6 -> 8
- net /SCR_RESET: track 0.00 -> 70.9 mm
- net /SPI.MOSI: track 29.5 -> 99.1 mm, vias 0 -> 2
- net /Keyboard/COL6: track 57.4 -> 125.9 mm, vias 7 -> 9
- net /Keyboard/ROW2: track 103.5 -> 171.0 mm, vias 0 -> 1
- net /Keyboard/COL8: track 65.3 -> 132.9 mm, vias 7 -> 9
- net /SPI.MISO: track 36.1 -> 103.6 mm, vias 0 -> 4
- net /SCR_CD: track 0.00 -> 67.2 mm
- net /GPS_EN: track 0.00 -> 66.0 mm, vias 0 -> 2
- net /SPI.SCK: track 32.7 -> 98.5 mm, vias 0 -> 5
- net /RXD0_ESP: track 0.00 -> 63.8 mm, vias 0 -> 2
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
Commit message: Finished PCB
Parts:
- added G***: LOGO, LOGO, F.Cu at (105.0, 143.0)
- added G***: LOGO, LOGO, F.Cu at (175.5, 144.5)
- added G***: LOGO, LOGO, B.Cu at (129.8, 35.2)
- added G***: LOGO, LOGO, B.Cu at (153.4, 35.2)
- added G***: LOGO, LOGO, B.Cu at (140.1, 114.0)
- added J2: Conn_02x05_Odd_Even, Connector_PinSocket_2.54mm:PinSocket_2x05_P2.54mm_Horizontal, B.Cu at (173.4, 54.9)
- added REF**: KiCad-Logo2_8mm_SilkScreen, Symbol:KiCad-Logo2_8mm_SilkScreen, F.Cu at (158.5, 35.5)
- added REF**: OSHW-Logo2_36.5x30mm_SilkScreen, Symbol:OSHW-Logo2_36.5x30mm_SilkScreen, B.Cu at (140.1, 144.0)
- moved C29 1.34 mm to (111.7, 80.4)
- moved C22 1.26 mm to (112.0, 79.1)
- moved REF** 1.04 mm to (140.2, 38.1)
- moved RF2 1.02 mm to (175.1, 33.4)
- moved RF1 1.02 mm to (105.0, 33.4)
- moved L2 0.67 mm to (175.1, 37.5), turned to 90 degrees
- moved R23 0.54 mm to (113.7, 97.2), turned to -90 degrees
- moved C31 0.39 mm to (111.6, 81.6)
- moved U1 0.26 mm to (140.0, 75.1)
Routing:
- net /IO38: track 0.00 -> 106.4 mm, vias 0 -> 3
- net /IO7: track 0.00 -> 97.3 mm, vias 0 -> 5
- net /IO5: track 0.00 -> 94.2 mm, vias 0 -> 3
- net /IO18: track 0.00 -> 90.8 mm, vias 0 -> 4
- net /IO6: track 0.00 -> 78.8 mm, vias 0 -> 4
- net GND: track 30.0 -> 100.5 mm, vias 54 -> 544
- net /IO2: track 0.00 -> 65.8 mm, vias 0 -> 3
- net /IO1: track 0.00 -> 61.0 mm, vias 0 -> 3
- net /3V3: track 316.7 -> 356.2 mm
- net +1V1: track 16.9 -> 45.5 mm, vias 0 -> 3
- net /Keyboard/XIN: track 20.3 -> 24.7 mm
- net /Keyboard/ROW4: track 172.9 -> 168.8 mm
- net /Keyboard/ROW1: track 151.6 -> 147.7 mm
- net /TCH_CS: track 59.1 -> 62.8 mm
- net /Keyboard/XOUT: track 20.2 -> 23.8 mm
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Other:
- board size 88.9 x 121.6 mm -> 90.8 x 121.7 mm
- board text added: "+ -"
- board text added: "3V3"
- board text added: "BEWARE OF THE MANUELA EFFECT"
- board text added: "BOOT"
- board text added: "CHARGING LEDS"
- board text added: "DESIGNED IN SPAIN"
- board text added: "EA9353URE"
- board text added: "GND"
- board text added: "IO1"
- board text added: "IO18"
- board text added: "IO2"
- board text added: "IO38"
- board text added: "IO5"
- board text added: "IO6"
- board text added: "IO7"
- board text added: "NO LE BUSQUES TRES PIES..."
- board text added: "POWER LEDS"
- board text added: "RESET"
- board text added: "SWCLK"
- board text added: "SWD"
- board text added: "by ThePangel"
- board text removed: "${REFERENCE}"
